File: PCB_Waschanlage.kicad_pcb (KiCad board)
At the start: 2 copper layers, 228 x 75 mm, 81 parts, among them J10 JMPR_LED_BTN_Sensor_1, J11 JMPR_LED_BTN_Sensor_4, J12 Conn_LED_Error, J13 Conn_LED_MainWash, J14 Conn_BTN_Start, J15 Conn_BTN_Basic, J16 Conn_LED_Motor, J17 Conn_LED_Red, J18 Conn_BTN_Sensor_1, J19 Conn_BTN_Sensor_4, J20 JMPR_LED_PreWash, J21 JMPR_LED_Start, J22 JMPR_LED_Basic, J23 JMPR_LED_BTN_On_Off, J24 JMPR_LED_BTN_Special, J25 JMPR_LED_Green, J26 JMPR_LED_BTN_Sensor_2, J27 JMPR_LED_BTN_Sensor_5, J28 Conn_LED_PreWash, J29 Conn_LED_Start, J3 Conn_Fuse, J30 Conn_LED_Basic, J31 Conn_BTN_On_Off, J32 Conn_BTN_Special, J33 Conn_LED_Green, J34 Conn_BTN_Sensor_2, J35 Conn_BTN_Sensor_5, J36 JMPR_LED_Special, J37 JMPR_LED_Care, J38 JMPR_LED_Underbody, J39 JMPR_LED_BTN_EmergencyOff, J4 JMPR_LED_Error, J40 JMPR_LED_BTN_Premium, J41 JMPR_LED_BTN_Sensor_3, J42 Conn_LED_Special, J43 Conn_LED_Care, J44 Conn_LED_Underbody, J45 Conn_BTN_EmergencyOff, J46 Conn_BTN_Premium, J47 Conn_BTN_Sensor_3, J48 JMPR_LED_Rims, J49 JMPR_LED_Premium, J5 JMPR_LED_MainWash, J50 JMPR_LED_Dry, J51 Conn_LED_Rims, J52 Conn_LED_Premium, J53 Conn_LED_Dry, J54 Conn_AdditionalPins_1, J55 Conn_AdditionalPins_2, J56 Conn_AdditionalPins_3, J57 5103308-6, J58 5103308-6, J6 JMPR_LED_BTN_Start, J7 JMPR_LED_BTN_Basic, J8 JMPR_LED_Motor, J9 JMPR_LED_Red

Commit message: all done
Parts:
- added H1: MountingHole, MountingHole:MountingHole_4.3mm_M4, F.Cu at (46.0, 67.0)
- added H2: MountingHole, MountingHole:MountingHole_4.3mm_M4, F.Cu at (263.0, 67.0)
- added H3: MountingHole, MountingHole:MountingHole_4.3mm_M4, F.Cu at (263.0, 128.0)
- added H4: MountingHole, MountingHole:MountingHole_4.3mm_M4, F.Cu at (46.0, 128.0)
- added H5: MountingHole, MountingHole:MountingHole_4.3mm_M4, F.Cu at (155.0, 128.0)
- added H6: MountingHole, MountingHole:MountingHole_4.3mm_M4, F.Cu at (155.0, 67.0)
Routing:
- net VCC_in: track 218.0 -> 220.2 mm
Other:
- outline, holes or cut-outs redrawn
